File: PCB_Design/PCB_Design.kicad_pcb (KiCad board)
At the start: 2 copper layers, 25 parts, among them J1 Conn_01x02_Female, J2 Conn_01x02_Female, J3 Conn_01x02_Male, M1 MNMOS, U1 TLP250, U2 ATA00B36S-L, U3 TL494

Commit message: started pcb design, looking good for a newbie
Parts:
- removed M1: MNMOS, Package_TO_SOT_THT:TO-220-3_Vertical
- removed R1: 150, Resistor_SMD:R_2512_6332Metric
- added Q1: Q_NMOS_DGS, Package_TO_SOT_THT:TO-220-3_Vertical, F.Cu at (75.7, 44.1)
- C2, R10, R11, R8: moved to B.Cu
- D1: footprint Package_TO_SOT_THT:TO-220-2_Vertical -> Package_TO_SOT_THT:TO-220-2_Horizontal_TabDown
- moved D1 140.7 mm to (48.4, 48.1)
- moved J1 125.8 mm to (33.9, 24.4), turned to 270 degrees
- moved J2 114.0 mm to (41.4, 70.9)
- moved D2 108.4 mm to (128.2, 25.3)
- moved U2 100.4 mm to (93.0, 74.8), turned to 90 degrees
- moved C1 99.7 mm to (134.7, 43.4), turned to 180 degrees
- moved R6 96.6 mm to (129.8, 47.1), turned to 180 degrees
- moved U1 85.3 mm to (99.1, 52.3), turned to 180 degrees
- moved R8 80.6 mm to (137.6, 55.0)
- moved R7 78.0 mm to (140.7, 47.1), turned to 180 degrees
- moved C2 70.9 mm to (128.3, 54.8), turned to 180 degrees
- moved D3 70.4 mm to (145.7, 35.0), turned to 90 degrees
- moved R5 69.1 mm to (148.8, 47.2), turned to 270 degrees
- moved R3 67.0 mm to (127.2, 42.5), turned to 180 degrees
- moved R2 62.9 mm to (142.5, 41.6)
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Connections:
- B1 pad 1: VCC -> Net-(B1-Pad1)
- B1 pad 2: (no net) -> Net-(B1-Pad2)
- B1 pad 3: (no net) -> VCC
- B1 pad 4: (no net) -> VCC
- B1 pad 5: (no net) -> Net-(B1-Pad5)
- B1 pad 6: (no net) -> Net-(B1-Pad6)
- C3 pad 2: Net-(B1-Pad~) -> Net-(B1-Pad5)
- D1 pad 2: Net-(B1-Pad~) -> Net-(B1-Pad2)
- D2 pad 1: Net-(B1-Pad~) -> Net-(B1-Pad6)
- D3 pad 1: Net-(B1-Pad~) -> Net-(B1-Pad5)
- J3 pad 1: Net-(B1-Pad~) -> Net-(B1-Pad5)
Routing:
- net GND: track 0.00 -> 246.0 mm
- net VCC: track 0.00 -> 179.7 mm
- net Net-(B1-Pad5): track 0.00 -> 125.3 mm
- net /Vout: track 0.00 -> 67.9 mm
- net +12V: track 0.00 -> 61.0 mm
- net /1IN+: track 0.00 -> 37.7 mm
- net Net-(U2-Pad9): track 0.00 -> 32.6 mm
- net Net-(U1-Pad3): track 0.00 -> 29.4 mm
- net Net-(D2-Pad2): track 0.00 -> 29.3 mm
- net GND1: track 0.00 -> 27.9 mm
- net Net-(U1-Pad2): track 0.00 -> 27.1 mm, vias 0 -> 1
- net Net-(C1-Pad1): track 0.00 -> 24.0 mm
- net Net-(B1-Pad6): track 0.00 -> 18.2 mm
- net /GATE: track 0.00 -> 17.0 mm
- net Net-(R4-Pad2): track 0.00 -> 15.7 mm
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
Commit message: pcb design completed
Parts:
- added R1: 150, Resistor_THT:R_Axial_DIN0309_L9.0mm_D3.2mm_P12.70mm_Horizontal, B.Cu at (109.2, 83.8)
- added R12: 4K, Resistor_THT:R_Axial_DIN0309_L9.0mm_D3.2mm_P12.70mm_Horizontal, F.Cu at (147.3, 108.0)
- added R13: 1K, Resistor_THT:R_Axial_DIN0309_L9.0mm_D3.2mm_P12.70mm_Horizontal, F.Cu at (146.1, 91.4)
- added R9: 0.2, Resistor_THT:R_Axial_DIN0309_L9.0mm_D3.2mm_P12.70mm_Horizontal, F.Cu at (162.5, 90.8)
- C1, C3, U2: moved to B.Cu
- R10, R11, R8: footprint Resistor_SMD:R_2512_6332Metric -> Resistor_THT:R_Axial_DIN0309_L9.0mm_D3.2mm_P12.70mm_Horizontal; moved to F.Cu
- R2, R3, R4, R5, R6, R7: footprint Resistor_SMD:R_2512_6332Metric -> Resistor_THT:R_Axial_DIN0309_L9.0mm_D3.2mm_P12.70mm_Horizontal
- moved J2 80.7 mm to (109.1, 114.7)
- moved J1 64.0 mm to (62.7, 81.5)
- moved R2 63.4 mm to (151.6, 104.3)
- moved R7 58.1 mm to (124.5, 102.9), turned to 0 degrees
- moved R5 56.2 mm to (124.5, 97.8), turned to 0 degrees
- moved R6 56.0 mm to (153.7, 97.8), turned to 0 degrees
- moved R8 53.5 mm to (109.2, 100.3)
- moved R11 53.0 mm to (142.2, 101.6)
- moved C3 50.7 mm to (195.6, 84.2)
- moved D1 48.4 mm to (72.2, 90.3)
- moved J3 48.3 mm to (207.0, 99.1)
- moved C1 47.0 mm to (127.5, 89.9), turned to 90 degrees
- moved R10 46.9 mm to (143.7, 85.8), turned to 0 degrees
- moved D2 46.5 mm to (144.7, 68.8), turned to 180 degrees
- moved L1 41.1 mm to (165.6, 68.9)
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Connections:
- net Net-(C1-Pad1) renamed /REF
- B1 pad 5: Net-(B1-Pad5) -> /2IN+
- C3 pad 2: Net-(B1-Pad5) -> /2IN+
- D1 pad 1: GND -> Net-(B1-Pad2)
- D1 pad 2: Net-(B1-Pad2) -> GND
- D2 pad 1: Net-(B1-Pad6) -> Net-(D2-Pad1)
- D2 pad 2: Net-(D2-Pad2) -> Net-(B1-Pad6)
- D3 pad 1: Net-(B1-Pad5) -> Net-(D2-Pad1)
- D3 pad 2: Net-(D2-Pad2) -> /2IN+
- J3 pad 1: Net-(B1-Pad5) -> /2IN+
- L1 pad 1: Net-(D2-Pad2) -> Net-(D2-Pad1)
- U3 pad 15: Net-(U3-Pad15) -> /2IN-
- U3 pad 16: Net-(U3-Pad16) -> /2IN+
Routing:
- net Net-(B1-Pad5): track 125.3 -> 0.00 mm
- net /2IN+: track 0.00 -> 122.8 mm
- net VCC: track 179.7 -> 99.4 mm
- net Net-(C1-Pad2): track 13.5 -> 53.5 mm
- net GND1: track 27.9 -> 58.6 mm
- net Net-(D2-Pad2): track 29.3 -> 0.00 mm
- net Net-(D2-Pad1): track 0.00 -> 26.0 mm
- net /1IN+: track 37.7 -> 13.2 mm
- net /2IN-: track 0.00 -> 20.5 mm
- net GND: track 246.0 -> 226.6 mm, vias 0 -> 1
- net +12V: track 61.0 -> 41.6 mm
- net /REF: track 24.0 -> 39.4 mm
- net Net-(R4-Pad1): track 13.8 -> 23.8 mm
- net Net-(R1-Pad2): track 32.6 -> 41.8 mm, vias 0 -> 1
- net Net-(B1-Pad2): track 14.5 -> 22.1 mm
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Other:
- board outline added: 162.6 x 73.7 mm
- board text added: "EE464 - Corona Semester 2020 Forward Converter Design by PowerLovers"

Commit message: design completed. gerber files and bom are added
Parts:
- D1: footprint Package_TO_SOT_THT:TO-220-2_Horizontal_TabDown -> Package_TO_SOT_SMD:TO-277A
- D2, D3: footprint Package_TO_SOT_THT:TO-220-2_Vertical -> Package_TO_SOT_SMD:TO-277A
- J3: value Conn_01x02_Male -> Conn_01x02_Female
- Q1: footprint Package_TO_SOT_THT:TO-220-3_Vertical -> Package_TO_SOT_SMD:PQFN_8x8
- R3: value 9.1K -> 8.2K
- moved J3 30.1 mm to (212.3, 69.4), turned to 270 degrees
- moved J1 5.56 mm to (63.7, 76.0)
- moved U1 2.62 mm to (102.3, 79.2)
- moved J2 0.47 mm to (109.4, 115.0)
Connections:
- J3 pad 1: /2IN+ -> /Vout
- J3 pad 2: /Vout -> /2IN+
Routing:
- net GND: track 226.6 -> 255.4 mm
- net VCC: track 99.4 -> 118.9 mm
- net /2IN+: track 122.8 -> 133.6 mm, vias 0 -> 1
- net Net-(B1-Pad6): track 19.4 -> 25.6 mm
- net /GATE: track 12.5 -> 18.7 mm
- net /Vout: track 71.8 -> 76.9 mm
- net Net-(B1-Pad2): track 22.1 -> 25.7 mm, vias 0 -> 1
- net Net-(U1-Pad3): track 27.0 -> 24.3 mm
- net GND1: track 58.6 -> 56.2 mm
- net +12V: track 41.6 -> 39.3 mm
- net Net-(R1-Pad1): track 21.3 -> 19.2 mm
- net Net-(B1-Pad1): track 8.88 -> 7.08 mm
- added copper zone on B.Cu, net GND
