File: PCB_Design/PCB_Design.sch (KiCad schematic (older format))
At the start: 28 parts, among them J1 Conn_01x02_Female, J2 Conn_01x02_Female, J3 Conn_01x02_Male, Q1 Q_NMOS_DGS, U1 TLP250, U2 ATA00B36S-L, U3 TL494

Commit message: design completed. gerber files and bom are added
Parts:
- removed J3: Conn_01x02_Male, Connector:Banana_Jack_2Pin, symbol Connector:Conn_01x02_Male
- added J3: Conn_01x02_Female, Connector:Banana_Jack_2Pin, symbol Connector:Conn_01x02_Female
- D1: footprint Package_TO_SOT_THT:TO-220-2_Horizontal_TabDown -> Package_TO_SOT_SMD:TO-277A
- D2, D3: footprint Package_TO_SOT_THT:TO-220-2_Vertical -> Package_TO_SOT_SMD:TO-277A
- Q1: footprint Package_TO_SOT_THT:TO-220-3_Vertical -> Package_TO_SOT_SMD:PQFN_8x8
- R3: value 9.1K -> 8.2K
Connections:
- net 2IN+: now also J3.2 (Pin_2)
- net Vout: now also J3.1 (Pin_1)
Changed lines of the file:
@@
 F 0 "D1" H 3300 4065 50  0000 C CNN
 F 1 "DIODE" H 3300 3974 50  0000 C CNN
-F 2 "Package_TO_SOT_THT:TO-220-2_Horizontal_TabDown" H 3300 3800 50  0001 C CNN
+F 2 "Package_TO_SOT_SMD:TO-277A" H 3300 3800 50  0001 C CNN
 F 3 "~" H 3300 3800 50  0001 C CNN
 	1    3300 3800
@@
 F 0 "D2" H 4550 3065 50  0000 C CNN
 F 1 "DIODE" H 4550 2974 50  0000 C CNN
-F 2 "Package_TO_SOT_THT:TO-220-2_Vertical" H 4550 2800 50  0001 C CNN
+F 2 "Package_TO_SOT_SMD:TO-277A" H 4550 2800 50  0001 C CNN
 F 3 "~" H 4550 2800 50  0001 C CNN
 	1    4550 2800
@@
 L power:PWR_FLAG #FLG0101
 U 1 1 5EEA4059
-P 2850 1000
-F 0 "#FLG0101" H 2850 1075 50  0001 C CNN
-F 1 "PWR_FLAG" H 2850 1173 50  0000 C CNN
-F 2 "" H 2850 1000 50  0001 C CNN
-F 3 "~" H 2850 1000 50  0001 C CNN
-	1    2850 1000
+P 9200 4350
+F 0 "#FLG0101" H 9200 4425 50  0001 C CNN
+F 1 "PWR_FLAG" H 9200 4523 50  0000 C CNN
+F 2 "" H 9200 4350 50  0001 C CNN
+F 3 "~" H 9200 4350 50  0001 C CNN
+	1    9200 4350
 	1    0    0    -1
 $EndComp
@@
 L power:PWR_FLAG #FLG0102
 U 1 1 5EEA6CC1
-P 3050 1300
-F 0 "#FLG0102" H 3050 1375 50  0001 C CNN
-F 1 "PWR_FLAG" H 3050 1473 50  0000 C CNN
-F 2 "" H 3050 1300 50  0001 C CNN
-F 3 "~" H 3050 1300 50  0001 C CNN
-	1    3050 1300
+P 9400 4650
+F 0 "#FLG0102" H 9400 4725 50  0001 C CNN
+F 1 "PWR_FLAG" H 9400 4823 50  0000 C CNN
+F 2 "" H 9400 4650 50  0001 C CNN
+F 3 "~" H 9400 4650 50  0001 C CNN
+	1    9400 4650
 	-1   0    0    1
 $EndComp
@@
 L power:PWR_FLAG #FLG0103
 U 1 1 5EECA3DB
-P 1500 1000
-F 0 "#FLG0103" H 1500 1075 50  0001 C CNN
-F 1 "PWR_FLAG" H 1500 1173 50  0000 C CNN
-F 2 "" H 1500 1000 50  0001 C CNN
-F 3 "~" H 1500 1000 50  0001 C CNN
-	1    1500 1000
+P 7850 4350
+F 0 "#FLG0103" H 7850 4425 50  0001 C CNN
+F 1 "PWR_FLAG" H 7850 4523 50  0000 C CNN
+F 2 "" H 7850 4350 50  0001 C CNN
+F 3 "~" H 7850 4350 50  0001 C CNN
+	1    7850 4350
 	1    0    0    -1
 $EndComp
@@
 L power:PWR_FLAG #FLG0104
 U 1 1 5EECCBFA
-P 1450 1350
-F 0 "#FLG0104" H 1450 1425 50  0001 C CNN
-F 1 "PWR_FLAG" H 1450 1523 50  0000 C CNN
-F 2 "" H 1450 1350 50  0001 C CNN
-F 3 "~" H 1450 1350 50  0001 C CNN
-	1    1450 1350
+P 7800 4700
+F 0 "#FLG0104" H 7800 4775 50  0001 C CNN
+F 1 "PWR_FLAG" H 7800 4873 50  0000 C CNN
+F 2 "" H 7800 4700 50  0001 C CNN
+F 3 "~" H 7800 4700 50  0001 C CNN
+	1    7800 4700
 	-1   0    0    1
 $EndComp
@@
 P 5950 4550
 F 0 "R3" V 6157 4550 50  0000 C CNN
-F 1 "9.1K" V 6066 4550 50  0000 C CNN
+F 1 "8.2K" V 6066 4550 50  0000 C CNN
 F 2 "Resistor_THT:R_Axial_DIN0309_L9.0mm_D3.2mm_P12.70mm_Horizontal" V 5880 4550 50  0001 C CNN
 F 3 "~" H 5950 4550 50  0001 C CNN
@@
 	5950 5650 5550 5650
 $Comp
-L Connector:Conn_01x02_Female J1
-U 1 1 5EED628F
-P 1550 1100
-F 0 "J1" H 1578 1076 50  0000 L CNN
-F 1 "Conn_01x02_Female" H 1578 985 50  0000 L CNN
-F 2 "Connector:Banana_Jack_2Pin" H 1550 1100 50  0001 C CNN
-F 3 "~" H 1550 1100 50  0001 C CNN
-	1    1550 1100
-	1    0    0    -1
-$EndComp
-$Comp
-L Connector:Conn_01x02_Female J2
-U 1 1 5EED6E52
-P 3050 1000
-F 0 "J2" H 3078 976 50  0000 L CNN
-F 1 "Conn_01x02_Female" H 3078 885 50  0000 L CNN
-F 2 "Connector:Banana_Jack_2Pin" H 3050 1000 50  0001 C CNN
-F 3 "~" H 3050 1000 50  0001 C CNN
-	1    3050 1000
-	1    0    0    -1
-$EndComp
-$Comp
 L power:VCC #PWR0117
 U 1 1 5EED7279
-P 1350 1100
-F 0 "#PWR0117" H 1350 950 50  0001 C CNN
-F 1 "VCC" H 1365 1273 50  0000 C CNN
-F 2 "" H 1350 1100 50  0001 C CNN
-F 3 "" H 1350 1100 50  0001 C CNN
-	1    1350 1100
+P 7700 4450
+F 0 "#PWR0117" H 7700 4300 50  0001 C CNN
+F 1 "VCC" H 7715 4623 50  0000 C CNN
+F 2 "" H 7700 4450 50  0001 C CNN
+F 3 "" H 7700 4450 50  0001 C CNN
+	1    7700 4450
 	1    0    0    -1
 $EndComp
@@
 L power:GND #PWR0118
 U 1 1 5EED7C06
-P 1350 1200
-F 0 "#PWR0118" H 1350 950 50  0001 C CNN
-F 1 "GND" H 1355 1027 50  0000 C CNN
-F 2 "" H 1350 1200 50  0001 C CNN
-F 3 "" H 1350 1200 50  0001 C CNN
-	1    1350 1200
+P 7700 4550
+F 0 "#PWR0118" H 7700 4300 50  0001 C CNN
+F 1 "GND" H 7705 4377 50  0000 C CNN
+F 2 "" H 7700 4550 50  0001 C CNN
+F 3 "" H 7700 4550 50  0001 C CNN
+	1    7700 4550
 	1    0    0    -1
 $EndComp
@@
 L power:+12V #PWR0119
 U 1 1 5EED7F95
-P 2850 1000
-F 0 "#PWR0119" H 2850 850 50  0001 C CNN
-F 1 "+12V" H 2865 1173 50  0000 C CNN
-F 2 "" H 2850 1000 50  0001 C CNN
-F 3 "" H 2850 1000 50  0001 C CNN
-	1    2850 1000
+P 9200 4350
+F 0 "#PWR0119" H 9200 4200 50  0001 C CNN
+F 1 "+12V" H 9215 4523 50  0000 C CNN
+F 2 "" H 9200 4350 50  0001 C CNN
+F 3 "" H 9200 4350 50  0001 C CNN
+	1    9200 4350
 	0    -1   -1   0
 $EndComp
@@
 L power:GND1 #PWR0120
 U 1 1 5EED8B6A
-P 2850 1100
-F 0 "#PWR0120" H 2850 850 50  0001 C CNN
-F 1 "GND1" H 2855 927 50  0000 C CNN
-F 2 "" H 2850 1100 50  0001 C CNN
-F 3 "" H 2850 1100 50  0001 C CNN
-	1    2850 1100
+P 9200 4450
+F 0 "#PWR0120" H 9200 4200 50  0001 C CNN
+F 1 "GND1" H 9205 4277 50  0000 C CNN
+F 2 "" H 9200 4450 50  0001 C CNN
+F 3 "" H 9200 4450 50  0001 C CNN
+	1    9200 4450
 	1    0    0    -1
 $EndComp
@@
 NoConn ~ 3150 5400
 Wire Wire Line
-	1500 1100 1350 1100
-Connection ~ 1350 1100
-Wire Wire Line
-	1450 1200 1350 1200
-Connection ~ 1350 1200
-Connection ~ 2850 1000
-Wire Wire Line
-	3050 1300 3050 1100
-Wire Wire Line
-	3050 1100 2850 1100
-Connection ~ 2850 1100
+	7850 4450 7700 4450
+Wire Wire Line
+	7800 4550 7700 4550
+Wire Wire Line
+	9400 4450 9200 4450
 Wire Wire Line
 	7600 3150 7150 3150
@@
 Wire Wire Line
 	7150 3250 7150 3600
-$Comp
-L Connector:Conn_01x02_Male J3
-U 1 1 5EEC8F4E
-P 7800 3250
-F 0 "J3" H 7772 3132 50  0000 R CNN
-F 1 "Conn_01x02_Male" H 7772 3223 50  0000 R CNN
-F 2 "Connector:Banana_Jack_2Pin" H 7800 3250 50  0001 C CNN
-F 3 "~" H 7800 3250 50  0001 C CNN
-	1    7800 3250
-	-1   0    0    1
-$EndComp
-Wire Wire Line
-	1500 1000 1500 1100
-Wire Wire Line
-	1450 1200 1450 1350
+Wire Wire Line
+	7850 4350 7850 4450
 Wire Wire Line
 	2650 4000 2750 4000
@@
 F 0 "Q1" H 2854 4246 50  0000 L CNN
 F 1 "Q_NMOS_DGS" H 2854 4155 50  0000 L CNN
-F 2 "Package_TO_SOT_THT:TO-220-3_Vertical" H 2850 4300 50  0001 C CNN
+F 2 "Package_TO_SOT_SMD:PQFN_8x8" H 2850 4300 50  0001 C CNN
 F 3 "~" H 2650 4200 50  0001 C CNN
 	1    2650 4200
@@
 F 0 "D3" V 5396 3072 50  0000 R CNN
 F 1 "DIODE" V 5305 3072 50  0000 R CNN
-F 2 "Package_TO_SOT_THT:TO-220-2_Vertical" H 5350 3200 50  0001 C CNN
+F 2 "Package_TO_SOT_SMD:TO-277A" H 5350 3200 50  0001 C CNN
 F 3 "~" H 5350 3200 50  0001 C CNN
 	1    5350 3200
@@
 NoConn ~ 4550 5250
 NoConn ~ 4550 4950
+Wire Wire Line
+	7800 4550 7800 4650
+Connection ~ 7800 4650
+Wire Wire Line
+	7800 4650 7800 4700
+Connection ~ 7850 4450
+Wire Wire Line
+	9600 4350 9200 4350
+Connection ~ 9200 4350
+$Comp
+L Connector:Conn_01x02_Female J1
+U 1 1 5EF0F034
+P 8400 4500
+F 0 "J1" H 8428 4476 50  0000 L CNN
+F 1 "Conn_01x02_Female" H 8428 4385 50  0000 L CNN
+F 2 "Connector:Banana_Jack_2Pin" H 8400 4500 50  0001 C CNN
+F 3 "~" H 8400 4500 50  0001 C CNN
+	1    8400 4500
+	1    0    0    -1
+$EndComp
+Wire Wire Line
+	8200 4450 8200 4500
+Wire Wire Line
+	7850 4450 8200 4450
+Wire Wire Line
+	8200 4650 8200 4600
+Wire Wire Line
+	7800 4650 8200 4650
+$Comp
+L Connector:Conn_01x02_Female J2
+U 1 1 5EF17833
+P 9800 4350
+F 0 "J2" H 9828 4326 50  0000 L CNN
+F 1 "Conn_01x02_Female" H 9828 4235 50  0000 L CNN
+F 2 "Connector:Banana_Jack_2Pin" H 9800 4350 50  0001 C CNN
+F 3 "~" H 9800 4350 50  0001 C CNN
+	1    9800 4350
+	1    0    0    -1
+$EndComp
+$Comp
+L Connector:Conn_01x02_Female J3
+U 1 1 5EF17F43
+P 7800 3150
+F 0 "J3" H 7828 3126 50  0000 L CNN
+F 1 "Conn_01x02_Female" H 7828 3035 50  0000 L CNN
+F 2 "Connector:Banana_Jack_2Pin" H 7800 3150 50  0001 C CNN
+F 3 "~" H 7800 3150 50  0001 C CNN
+	1    7800 3150
+	1    0    0    -1
+$EndComp
+Wire Wire Line
+	9400 4450 9400 4650
+Wire Wire Line
+	9600 4450 9400 4450
+Connection ~ 9400 4450
 $EndSCHEMATC
